File: kicad/Ki5.kicad_pcb (KiCad board)
At the start: 2 copper layers, 90 x 120 mm, 542 parts, among them IC1 VSC8541XMV-01, J1 Conn_02x20_Odd_Even, J10 Micro_SD_Card_Det, J11 Conn_02x05_Odd_Even, J12 RJHSE5384, J13 Conn_02x04_Odd_Even, J14 Conn_02x11_Odd_Even, J15 Conn_Coaxial, J16 Conn_Coaxial, J17 Conn_Coaxial, J18 Conn_Coaxial, J19 Fan_Tacho, J2 Conn_02x10_Odd_Even, J3 Conn_Coaxial, J4 Conn_Coaxial, J5 Conn_Coaxial, J6 Conn_Coaxial, J7 USB_B_Micro, J8 Jack-DC, J9 ASP-134602-01, M1 Mounting_Hole_PAD, M2 Mounting_Hole_PAD, M3 Mounting_Hole_PAD, M4 Mounting_Hole_PAD, M5 Mounting_Hole_PAD, M6 Mounting_Hole_PAD, Q1 FDG6335N, Q2 FDG6335N, Q4 FDG6335N, Q5 FDG6335N, Q6 IRLML6402, T1 TG111-MSC13LF, U1 FU540-C000, U10 H5AN8G8NAFR-UH, U11 TPS51200DRC, U12 IS25WP256D, U13 FT2232HL, U14 TLV62080DSGx, U15 TLV62084DSGx, U16 TLV62095RGTR, U17 LP5907MFX-1.8/NOPB, U18 TPS51363, U19 LM3880MFE-1AA/NOPB, U2 H5AN8G8NAFR-UH, U20 SN74AUP1T34DCKR, U21 SN74AUP1T34DCKR, U22 SN74AUP1T34DCKR, U23 SN74AUP1T34DCKR, U24 SN74AUP1T34DCKR, U25 SN74AUP1T34DCKR, U26 TPD6F003, U27 TPS62133RGTT, U28 SN74AUP1T34DCKR, U29 SN74AUP1T34DCKR, U3 H5AN8G8NAFR-UH, U30 SN74AUP1T34DCKR, U31 SN74AUP1T34DCKR, U32 SN74AUP1T34DCKR, U33 SN74AUP1T34DCKR, U35 MIC5353-2.5YMT-TR, U36 NCP133AMX100TCG, U37 SN74AUP1T34DCKR, U38 SN74AUP1T34DCKR, U4 H5AN8G8NAFR-UH, U49 M24C02-WMN, U5 H5AN8G8NAFR-UH, U50 TLV62080DSGx, U6 H5AN8G8NAFR-UH, U7 H5AN8G8NAFR-UH, U8 H5AN8G8NAFR-UH, U9 H5AN8G8NAFR-UH, X1 33.3333 MHz, X2 1.0 MHz, Y1 33.333 MHz, Y2 12 MHz, Y3 25 MHz

Commit message: Updated for 3D
Parts:
- J8: footprint Connector_BarrelJack:BarrelJack_CUI_PJ-063BH_Horizontal -> Connector_BarrelJack:BarrelJack_CUI_PJ-063AH_Horizontal
- J9: footprint Connector_Samtec:Samtec_FMC_ASP-134602-01_10x40_P0.5mm_Vertical -> Connector_Samtec:Samtec_FMC_ASP-134602-01_10x40_P1.27mm_Vertical
- U18: footprint Package_DFN_QFN:R-VFQFN-28-1EP_3.5x4.5mm_P0.4mm_EP2.1x3.1mm -> Package_DFN_QFN:Texas_R-VFQFN-28-1EP_3.5x4.5mm_P0.4mm_EP2.1x3.1mm
- U26: footprint Package_SON:WSON-12-1EP_1.35x2.5mm_P0.4mm_EP0.4x2mm -> Package_SON:Texas_R-PWSON-N12_EP0.4x2mm
Other:
- board text added: "ki5 Board"

Commit message: Update kicad electric lines
Parts:
- added ?: MountingHole_2.7mm_M2.5_ISO7380_Pad, MountingHole:MountingHole_2.7mm_M2.5_ISO7380_Pad, F.Cu at (59.4, 69.9)
- added ?: MountingHole_2.7mm_M2.5_ISO7380_Pad, MountingHole:MountingHole_2.7mm_M2.5_ISO7380_Pad, F.Cu at (93.4, 69.9)
- added ?: MountingHole_2.7mm_M2.5_ISO7380_Pad, MountingHole:MountingHole_2.7mm_M2.5_ISO7380_Pad, F.Cu at (93.4, 103.9)
- added ?: MountingHole_2.7mm_M2.5_ISO7380_Pad, MountingHole:MountingHole_2.7mm_M2.5_ISO7380_Pad, F.Cu at (59.4, 103.9)
- moved R13 56.3 mm to (40.3, 87.6)
- moved R14 56.3 mm to (40.3, 89.2)
- moved D10 2.93 mm to (92.1, 134.9), turned to 90 degrees
- moved R72 1.25 mm to (95.2, 133.7), turned to 90 degrees
- moved C261 1.17 mm to (72.7, 102.0)
- moved C284 1.17 mm to (75.3, 101.5)
- moved R170 1.17 mm to (64.0, 103.3)
- moved C259 1.17 mm to (66.9, 103.3)
- moved C260 1.17 mm to (70.5, 102.0)
- moved C264 1.17 mm to (68.1, 102.0)
- moved C265 1.17 mm to (64.5, 102.0)
- moved R164 1.17 mm to (68.6, 103.5)
- moved R166 1.17 mm to (71.1, 103.5)
- moved R168 1.17 mm to (73.6, 103.5)
- moved R171 1.17 mm to (64.9, 103.3)
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Connections:
- C1 pad 1: Earth -> AGND
- C10 pad 1: Earth -> AGND
- C100 pad 1: Earth -> AGND
- C101 pad 1: Earth -> AGND
- C102 pad 1: Earth -> AGND
- C103 pad 1: Earth -> AGND
- C104 pad 1: Earth -> AGND
- C105 pad 1: Earth -> AGND
- C106 pad 1: Earth -> AGND
- C107 pad 1: Earth -> AGND
- C108 pad 1: Earth -> AGND
- C109 pad 1: Earth -> AGND
- C11 pad 1: Earth -> AGND
- C110 pad 1: Earth -> AGND
- C111 pad 1: Earth -> AGND
- C112 pad 1: Earth -> AGND
- C113 pad 1: Earth -> AGND
- C114 pad 1: Earth -> AGND
- C115 pad 1: Earth -> AGND
- C116 pad 1: Earth -> AGND
- C117 pad 1: Earth -> AGND
- C118 pad 1: Earth -> AGND
- C119 pad 1: Earth -> AGND
- C12 pad 1: Earth -> AGND
- C120 pad 1: Earth -> AGND
- C121 pad 1: Earth -> AGND
- C122 pad 1: Earth -> AGND
- C124 pad 1: Earth -> AGND
- C125 pad 2: Earth -> AGND
- C126 pad 2: Earth -> AGND
- C127 pad 2: Earth -> AGND
- C128 pad 2: Earth -> AGND
- C129 pad 2: Earth -> AGND
- C13 pad 1: Earth -> AGND
- C130 pad 2: Earth -> AGND
- C131 pad 2: Earth -> AGND
- C132 pad 2: Earth -> AGND
- C133 pad 2: Earth -> AGND
- C134 pad 1: Earth -> AGND
- C135 pad 1: Earth -> AGND
- C136 pad 1: Earth -> AGND
- C137 pad 1: Earth -> AGND
- C138 pad 1: Earth -> AGND
- C139 pad 1: Earth -> AGND
- C14 pad 1: Earth -> AGND
- C140 pad 1: Earth -> AGND
- C141 pad 1: Earth -> AGND
- C143 pad 2: Earth -> AGND
- C144 pad 2: Earth -> AGND
- C145 pad 2: Earth -> AGND
- C147 pad 1: Earth -> AGND
- C148 pad 1: Earth -> AGND
- C149 pad 1: Earth -> AGND
- C15 pad 1: Earth -> AGND
- C150 pad 2: Earth -> AGND
- C151 pad 2: Earth -> AGND
- C152 pad 1: Earth -> AGND
- C153 pad 2: Earth -> AGND
- C154 pad 2: Earth -> AGND
- C155 pad 2: Earth -> AGND
- C156 pad 2: Earth -> AGND
- C157 pad 2: Earth -> AGND
- C158 pad 2: Earth -> AGND
- C159 pad 2: Earth -> AGND
- C16 pad 1: Earth -> AGND
- C160 pad 2: Earth -> AGND
- C161 pad 2: Earth -> AGND
- C162 pad 2: Earth -> AGND
- C163 pad 1: Earth -> AGND
- C164 pad 2: Earth -> AGND
- C165 pad 2: Earth -> AGND
- C166 pad 1: Earth -> AGND
- C167 pad 1: Earth -> AGND
- C168 pad 1: Earth -> AGND
- C169 pad 1: Earth -> AGND
- C17 pad 1: Earth -> AGND
- C170 pad 1: Earth -> AGND
- C171 pad 1: Earth -> AGND
- C172 pad 1: Earth -> AGND
- C173 pad 1: Earth -> AGND
- C174 pad 1: Earth -> AGND
- C175 pad 1: Earth -> AGND
- C176 pad 1: Earth -> AGND
- C177 pad 1: Earth -> AGND
- C178 pad 2: Earth -> AGND
- C179 pad 2: Earth -> AGND
- C18 pad 1: Earth -> AGND
- C180 pad 1: Earth -> AGND
- C181 pad 2: Earth -> AGND
- C182 pad 2: Earth -> AGND
- C183 pad 2: Earth -> AGND
- C184 pad 1: Earth -> AGND
- C185 pad 1: Earth -> AGND
- C186 pad 2: Earth -> AGND
- C187 pad 1: Earth -> AGND
- C188 pad 2: Earth -> AGND
- C189 pad 2: Earth -> AGND
- C19 pad 1: Earth -> AGND
- C190 pad 2: Earth -> AGND
- C191 pad 2: Earth -> AGND
- C192 pad 2: Earth -> AGND
- C193 pad 2: Earth -> AGND
- C194 pad 2: Earth -> AGND
- C195 pad 2: Earth -> AGND
- C196 pad 1: Earth -> AGND
- C197 pad 1: Earth -> AGND
- C198 pad 1: Earth -> AGND
- C199 pad 1: Earth -> AGND
- C199 pad 2: /Ethernet/P0_D2_N -> Net-(C199-Pad2)
- C2 pad 1: Earth -> AGND
- C20 pad 1: Earth -> AGND
- C200 pad 1: Earth -> AGND
- C201 pad 1: Earth -> AGND
- C202 pad 1: Earth -> AGND
- C203 pad 1: Earth -> AGND
- C203 pad 2: Earth -> AGND
- C204 pad 1: Earth -> AGND
- C205 pad 2: Earth -> AGND
- C206 pad 1: Earth -> AGND
- C207 pad 1: Earth -> AGND
- C208 pad 2: Earth -> AGND
- C209 pad 1: Earth -> AGND
- C21 pad 1: Earth -> AGND
- C210 pad 1: Earth -> AGND
- C211 pad 1: Earth -> AGND
- C212 pad 1: Earth -> AGND
- C213 pad 2: Earth -> AGND
- C214 pad 2: Earth -> AGND
- C215 pad 2: Earth -> AGND
- C216 pad 2: Earth -> AGND
- C217 pad 2: Earth -> AGND
- C218 pad 1: Earth -> AGND
- C219 pad 1: Earth -> AGND
- C22 pad 1: Earth -> AGND
- C220 pad 1: Earth -> AGND
- C23 pad 1: Earth -> AGND
- C24 pad 1: Earth -> AGND
- C240 pad 1: Earth -> AGND
- C240 pad 2: Net-(C240-Pad2) -> VDD_DDR_VPP_N
- C241 pad 2: Earth -> AGND
- C242 pad 1: Earth -> AGND
- C243 pad 2: Earth -> AGND
- C244 pad 2: Earth -> AGND
- C245 pad 2: Earth -> AGND
- C246 pad 2: Earth -> AGND
- C247 pad 2: Earth -> AGND
- C248 pad 2: Earth -> AGND
- C249 pad 2: Earth -> AGND
- C25 pad 1: Earth -> AGND
- C250 pad 2: Earth -> AGND
- C251 pad 2: Earth -> AGND
- C252 pad 2: Earth -> AGND
- C253 pad 2: Earth -> AGND
- C254 pad 2: Earth -> AGND
- C255 pad 2: Earth -> AGND
- C256 pad 2: Earth -> AGND
- C257 pad 2: Earth -> AGND
- C258 pad 2: Earth -> AGND
- C259 pad 1: Earth -> AGND
- C26 pad 1: Earth -> AGND
- C260 pad 1: Earth -> AGND
- C261 pad 1: Earth -> AGND
- C262 pad 1: Earth -> AGND
- C263 pad 1: Earth -> AGND
- C264 pad 1: Earth -> AGND
- C265 pad 1: Earth -> AGND
- C267 pad 1: Earth -> AGND
- C268 pad 1: Earth -> AGND
- C268 pad 2: Net-(C240-Pad2) -> VDD_DDR_VPP_N
- C269 pad 1: Earth -> AGND
- C27 pad 1: Earth -> AGND
- C270 pad 1: Earth -> AGND
- C271 pad 1: Earth -> AGND
- C272 pad 1: Earth -> AGND
- C273 pad 1: Earth -> AGND
- C274 pad 1: Earth -> AGND
- C275 pad 1: Earth -> AGND
- C276 pad 1: Earth -> AGND
- C277 pad 1: Earth -> AGND
- C278 pad 1: Earth -> AGND
- C279 pad 1: Earth -> AGND
- C28 pad 1: Earth -> AGND
- C280 pad 1: Earth -> AGND
- C281 pad 1: Earth -> AGND
- C284 pad 1: Earth -> AGND
- C29 pad 1: Earth -> AGND
- C3 pad 1: Earth -> AGND
- C30 pad 1: Earth -> AGND
- C31 pad 1: Earth -> AGND
- C32 pad 1: Earth -> AGND
- C33 pad 1: Earth -> AGND
- C34 pad 1: Earth -> AGND
- C35 pad 1: Earth -> AGND
- C36 pad 1: Earth -> AGND
- C37 pad 1: Earth -> AGND
- C38 pad 1: Earth -> AGND
- C39 pad 1: Earth -> AGND
- C4 pad 1: Earth -> AGND
- C40 pad 1: Earth -> AGND
- C41 pad 1: Earth -> AGND
- C42 pad 1: Earth -> AGND
- C43 pad 1: Earth -> AGND
- C44 pad 2: Earth -> AGND
- C45 pad 1: Earth -> AGND
- C46 pad 1: Earth -> AGND
- C47 pad 1: Earth -> AGND
- C48 pad 1: Earth -> AGND
- C49 pad 1: Earth -> AGND
- C5 pad 1: Earth -> AGND
- C50 pad 1: Earth -> AGND
- C51 pad 1: Earth -> AGND
- C52 pad 1: Earth -> AGND
- C53 pad 1: Earth -> AGND
- C54 pad 1: Earth -> AGND
- C55 pad 1: Earth -> AGND
- C56 pad 1: Earth -> AGND
- C57 pad 1: Earth -> AGND
- C58 pad 1: Earth -> AGND
- C59 pad 1: Earth -> AGND
- C6 pad 1: Earth -> AGND
- C60 pad 1: Earth -> AGND
- C61 pad 1: Earth -> AGND
- C62 pad 1: Earth -> AGND
- C63 pad 1: Earth -> AGND
- C64 pad 1: Earth -> AGND
- C65 pad 1: Earth -> AGND
- C66 pad 1: Earth -> AGND
- C67 pad 1: Earth -> AGND
- C68 pad 1: Earth -> AGND
- C69 pad 1: Earth -> AGND
- C7 pad 1: Earth -> AGND
- C70 pad 1: Earth -> AGND
- C71 pad 1: Earth -> AGND
- C72 pad 1: Earth -> AGND
- C73 pad 1: Earth -> AGND
- C74 pad 1: Earth -> AGND
- C75 pad 1: Earth -> AGND
- C76 pad 1: Earth -> AGND
- C77 pad 1: Earth -> AGND
- C78 pad 1: Earth -> AGND
- C79 pad 1: Earth -> AGND
- C8 pad 1: Earth -> AGND
- C80 pad 1: Earth -> AGND
- C81 pad 1: Earth -> AGND
- C82 pad 1: Earth -> AGND
- C83 pad 1: Earth -> AGND
- C84 pad 1: Earth -> AGND
- C85 pad 1: Earth -> AGND
- C86 pad 1: Earth -> AGND
- C87 pad 1: Earth -> AGND
- C88 pad 1: Net-(C88-Pad1) -> /DDR4_x8_32b_1/REFIN
- C88 pad 2: Earth -> AGND
- C89 pad 1: Earth -> AGND
- C9 pad 1: Earth -> AGND
- C90 pad 1: Earth -> AGND
- C91 pad 1: Earth -> AGND
- C92 pad 1: Earth -> AGND
- C93 pad 1: Earth -> AGND
- C94 pad 2: Earth -> AGND
- C95 pad 2: Earth -> AGND
- C96 pad 2: Earth -> AGND
- C97 pad 2: Earth -> AGND
- C98 pad 2: Earth -> AGND
- C99 pad 2: Earth -> AGND
- D10 pad 1: Earth -> AGND
- D11 pad 1: Earth -> AGND
- D12 pad 1: Earth -> AGND
- D5 pad 1: Earth -> AGND
- D6 pad 1: Earth -> AGND
- D8 pad 2: Earth -> AGND
- D9 pad 1: Earth -> AGND
- IC1 pad 3: /Ethernet/P0_D2_N -> /Ethernet/P0_D3_N
- IC1 pad 4: /Ethernet/P0_D2_N -> /Ethernet/P0_D3_P
- IC1 pad 69: Earth -> AGND
- J1 pad 1: Earth -> AGND
- J1 pad 10: /Freedom-U540_2/QSPI1_DQ1_R -> /Freedom-U540_2/GPIO9
- J1 pad 11: /Freedom-U540_2/UART1_TX -> /Freedom-U540_2/GPIO6
- J1 pad 12: /Freedom-U540_2/QSPI1_CS0_R -> /Freedom-U540_2/GPIO7
- J1 pad 13: /Freedom-U540_2/UART1_RX -> /Freedom-U540_2/GPIO4
- J1 pad 14: /Freedom-U540_2/QSPI1_DQ0_R -> /Freedom-U540_2/GPIO5
- J1 pad 15: /Freedom-U540_2/I2C0_SCL -> /Freedom-U540_2/GPIO2
- J1 pad 16: Net-(J1-Pad16) -> /Freedom-U540_2/GPIO3
- J1 pad 17: /Freedom-U540_2/I2C0_SDA -> /Freedom-U540_2/GPIO0
- J1 pad 18: Net-(J1-Pad18) -> /Freedom-U540_2/GPIO1
- J1 pad 2: Earth -> AGND
- J1 pad 23: /Freedom-U540_2/GPIO0 -> /Freedom-U540_2/I2C0_SDA
- J1 pad 24: /Freedom-U540_2/GPIO1 -> Net-(J1-Pad24)
- J1 pad 25: /Freedom-U540_2/GPIO2 -> /Freedom-U540_2/I2C0_SCL
- J1 pad 26: /Freedom-U540_2/GPIO3 -> Net-(J1-Pad26)
- J1 pad 27: /Freedom-U540_2/GPIO4 -> /Freedom-U540_2/UART1_RX
- J1 pad 28: /Freedom-U540_2/GPIO5 -> /Freedom-U540_2/QSPI1_DQ0_R
- J1 pad 29: /Freedom-U540_2/GPIO6 -> /Freedom-U540_2/UART1_TX
- J1 pad 3: Net-(J1-Pad3) -> +5V
- J1 pad 30: /Freedom-U540_2/GPIO7 -> /Freedom-U540_2/QSPI1_CS0_R
- J1 pad 31: /Freedom-U540_2/GPIO8 -> Net-(J1-Pad31)
- J1 pad 32: /Freedom-U540_2/GPIO9 -> /Freedom-U540_2/QSPI1_DQ1_R
- J1 pad 33: /Freedom-U540_2/GPIO15 -> UART0_RX
- J1 pad 34: Net-(J1-Pad34) -> /Freedom-U540_2/QSPI1_SCK_R
- J1 pad 35: VDD_GIVDD_P -> UART0_TX
- J1 pad 36: +12V -> RESET_N
- J1 pad 37: +5V -> Net-(J1-Pad37)
- J1 pad 38: +12V -> PWR_BTN_N
- J1 pad 39: Earth -> AGND
- J1 pad 4: PWR_BTN_N -> +12V
- J1 pad 40: Earth -> AGND
- J1 pad 5: UART0_TX -> VDD_GIVDD_P
- J1 pad 6: RESET_N -> +12V
- J1 pad 7: UART0_RX -> /Freedom-U540_2/GPIO15
- J1 pad 8: /Freedom-U540_2/QSPI1_SCK_R -> Net-(J1-Pad8)
- J1 pad 9: Net-(J1-Pad9) -> /Freedom-U540_2/GPIO8
- J10 pad 10: Earth -> AGND
- J10 pad 11: Earth -> AGND
- J10 pad 6: Earth -> AGND
- J11 pad 10: Earth -> AGND
- J11 pad 2: Earth -> AGND
- J12 pad 2: /Ethernet/MX3_N -> /Ethernet/MX4_P
- J12 pad SH: Earth -> AGND
- J13 pad 8: Earth -> AGND
- J14 pad 21: Earth -> AGND
- J14 pad 22: Earth -> AGND
- J15 pad 2: Earth -> AGND
- J16 pad 2: Earth -> AGND
- J17 pad 2: Earth -> AGND
- J18 pad 2: Earth -> AGND
- J19 pad 3: Earth -> AGND
- J2 pad 1: /Freedom-U540_2/PWM0_0 -> /Freedom-U540_2/PWM0_2
- J2 pad 10: /Freedom-U540_2/QSPI1_CS1_R -> /Freedom-U540_2/EN_VDD_SD
- J2 pad 11: /Freedom-U540_2/SD_CD -> /Freedom-U540_2/QSPI1_CS2_R
- J2 pad 12: /Freedom-U540_2/QSPI1_CS2_R -> /Freedom-U540_2/SD_CD
- J2 pad 13: Net-(J2-Pad13) -> /Freedom-U540_2/QSPI1_CS3_R
- J2 pad 14: /Freedom-U540_2/QSPI1_CS3_R -> Net-(J2-Pad14)
- J2 pad 15: /Freedom-U540_2/PWM1_0 -> AGND
- J2 pad 16: Earth -> /Freedom-U540_2/PWM1_0
- J2 pad 17: /Freedom-U540_2/PWM1_1 -> /Freedom-U540_2/PWM1_2
- J2 pad 18: /Freedom-U540_2/PWM1_2 -> /Freedom-U540_2/PWM1_1
- J2 pad 19: Earth -> /Freedom-U540_2/PWM1_3
- J2 pad 2: /Freedom-U540_2/PWM0_2 -> /Freedom-U540_2/PWM0_0
- J2 pad 20: /Freedom-U540_2/PWM1_3 -> AGND
- J2 pad 3: /Freedom-U540_2/PWM0_1 -> /Freedom-U540_2/PWM0_3
- J2 pad 4: /Freedom-U540_2/PWM0_3 -> /Freedom-U540_2/PWM0_1
- J2 pad 5: GEMGXL_RST -> /Freedom-U540_2/QSPI1_DQ2_R
- J2 pad 6: /Freedom-U540_2/QSPI1_DQ2_R -> GEMGXL_RST
- J2 pad 7: FASTLINK_FAIL -> /Freedom-U540_2/QSPI1_DQ3_R
- J2 pad 8: /Freedom-U540_2/QSPI1_DQ3_R -> FASTLINK_FAIL
- J2 pad 9: /Freedom-U540_2/EN_VDD_SD -> /Freedom-U540_2/QSPI1_CS1_R
- J3 pad 2: Earth -> AGND
- J4 pad 2: Earth -> AGND
- J5 pad 2: Earth -> AGND
- J6 pad 2: Earth -> AGND
- J7 pad 5: Earth -> AGND
- J7 pad 6: Earth -> AGND
- J8 pad 2: Earth -> AGND
- J9 pad A1: Earth -> AGND
- J9 pad A12: Earth -> AGND
- J9 pad A13: Earth -> AGND
- J9 pad A16: Earth -> AGND
- J9 pad A17: Earth -> AGND
- J9 pad A20: Earth -> AGND
- J9 pad A21: Earth -> AGND
- J9 pad A24: Earth -> AGND
- J9 pad A25: Earth -> AGND
- J9 pad A28: Earth -> AGND
- J9 pad A29: Earth -> AGND
- J9 pad A32: Earth -> AGND
- J9 pad A33: Earth -> AGND
- J9 pad A36: Earth -> AGND
- J9 pad A37: Earth -> AGND
- J9 pad A4: Earth -> AGND
- J9 pad A40: Earth -> AGND
- J9 pad A5: Earth -> AGND
- J9 pad A8: Earth -> AGND
- J9 pad A9: Earth -> AGND
- J9 pad B10: Earth -> AGND
- J9 pad B11: Earth -> AGND
- J9 pad B14: Earth -> AGND
- J9 pad B15: Earth -> AGND
- J9 pad B18: Earth -> AGND
- J9 pad B19: Earth -> AGND
- J9 pad B2: Earth -> AGND
- J9 pad B22: Earth -> AGND
- J9 pad B23: Earth -> AGND
- J9 pad B26: Earth -> AGND
- J9 pad B27: Earth -> AGND
- J9 pad B3: Earth -> AGND
- J9 pad B30: Earth -> AGND
- J9 pad B31: Earth -> AGND
- J9 pad B34: Earth -> AGND
- J9 pad B35: Earth -> AGND
- J9 pad B38: Earth -> AGND
- J9 pad B39: Earth -> AGND
- J9 pad B6: Earth -> AGND
- J9 pad B7: Earth -> AGND
- J9 pad C1: Earth -> AGND
- J9 pad C12: Earth -> AGND
- J9 pad C13: Earth -> AGND
- J9 pad C16: Earth -> AGND
- J9 pad C17: Earth -> AGND
- J9 pad C20: Earth -> AGND
- J9 pad C21: Earth -> AGND
- J9 pad C24: Earth -> AGND
- J9 pad C25: Earth -> AGND
- J9 pad C28: Earth -> AGND
- J9 pad C29: Earth -> AGND
- J9 pad C32: Earth -> AGND
- J9 pad C33: Earth -> AGND
- J9 pad C36: Earth -> AGND
- J9 pad C38: Earth -> AGND
- J9 pad C4: Earth -> AGND
- J9 pad C40: Earth -> AGND
- J9 pad C5: Earth -> AGND
- J9 pad C8: Earth -> AGND
- J9 pad C9: Earth -> AGND
- J9 pad D10: Earth -> AGND
- J9 pad D13: Earth -> AGND
- J9 pad D16: Earth -> AGND
- J9 pad D19: Earth -> AGND
- J9 pad D2: Earth -> AGND
- J9 pad D22: Earth -> AGND
- J9 pad D25: Earth -> AGND
- J9 pad D28: Earth -> AGND
- J9 pad D3: Earth -> AGND
- J9 pad D37: Earth -> AGND
- J9 pad D39: Earth -> AGND
- J9 pad D6: Earth -> AGND
- J9 pad D7: Earth -> AGND
- J9 pad E1: Earth -> AGND
- J9 pad E11: Earth -> AGND
- J9 pad E14: Earth -> AGND
- J9 pad E17: Earth -> AGND
- J9 pad E20: Earth -> AGND
- J9 pad E23: Earth -> AGND
- J9 pad E26: Earth -> AGND
- J9 pad E29: Earth -> AGND
- J9 pad E32: Earth -> AGND
- J9 pad E35: Earth -> AGND
- J9 pad E38: Earth -> AGND
- J9 pad E4: Earth -> AGND
- J9 pad E40: Earth -> AGND
- J9 pad E5: Earth -> AGND
- J9 pad E8: Earth -> AGND
- J9 pad F12: Earth -> AGND
- J9 pad F15: Earth -> AGND
- J9 pad F18: Earth -> AGND
- J9 pad F2: Earth -> AGND
- J9 pad F21: Earth -> AGND
- J9 pad F24: Earth -> AGND
- J9 pad F27: Earth -> AGND
- J9 pad F3: Earth -> AGND
- J9 pad F30: Earth -> AGND
- J9 pad F33: Earth -> AGND
- J9 pad F36: Earth -> AGND
- J9 pad F39: Earth -> AGND
- J9 pad F6: Earth -> AGND
- J9 pad F9: Earth -> AGND
- J9 pad G1: Earth -> AGND
- J9 pad G11: Earth -> AGND
- J9 pad G14: Earth -> AGND
- J9 pad G17: Earth -> AGND
- J9 pad G20: Earth -> AGND
- J9 pad G23: Earth -> AGND
- J9 pad G26: Earth -> AGND
- J9 pad G29: Earth -> AGND
- J9 pad G32: Earth -> AGND
- J9 pad G35: Earth -> AGND
- J9 pad G38: Earth -> AGND
- J9 pad G4: Earth -> AGND
- J9 pad G40: Earth -> AGND
- J9 pad G5: Earth -> AGND
- J9 pad G8: Earth -> AGND
- J9 pad H12: Earth -> AGND
- J9 pad H15: Earth -> AGND
- J9 pad H18: Earth -> AGND
- J9 pad H2: Earth -> AGND
- J9 pad H21: Earth -> AGND
- J9 pad H24: Earth -> AGND
- J9 pad H27: Earth -> AGND
- J9 pad H3: Earth -> AGND
- J9 pad H30: Earth -> AGND
- J9 pad H33: Earth -> AGND
- J9 pad H36: Earth -> AGND
- J9 pad H39: Earth -> AGND
- J9 pad H6: Earth -> AGND
- J9 pad H9: Earth -> AGND
- J9 pad J1: Earth -> AGND
- J9 pad J11: Earth -> AGND
- J9 pad J14: Earth -> AGND
- J9 pad J17: Earth -> AGND
- J9 pad J20: Earth -> AGND
- J9 pad J23: Earth -> AGND
- J9 pad J26: Earth -> AGND
- J9 pad J29: Earth -> AGND
- J9 pad J32: Earth -> AGND
- J9 pad J35: Earth -> AGND
- J9 pad J38: Earth -> AGND
- J9 pad J4: Earth -> AGND
- J9 pad J40: Earth -> AGND
- J9 pad J5: Earth -> AGND
- J9 pad J8: Earth -> AGND
- J9 pad K12: Earth -> AGND
- J9 pad K15: Earth -> AGND
- J9 pad K18: Earth -> AGND
- J9 pad K2: Earth -> AGND
- J9 pad K21: Earth -> AGND
- J9 pad K24: Earth -> AGND
- J9 pad K27: Earth -> AGND
- J9 pad K3: Earth -> AGND
- J9 pad K30: Earth -> AGND
- J9 pad K33: Earth -> AGND
- J9 pad K36: Earth -> AGND
- J9 pad K39: Earth -> AGND
- J9 pad K6: Earth -> AGND
- J9 pad K9: Earth -> AGND
- M1 pad 1: Earth -> AGND
- M2 pad 1: Earth -> AGND
- M3 pad 1: Earth -> AGND
- M4 pad 1: Earth -> AGND
- M5 pad 1: Earth -> AGND
- M6 pad 1: Earth -> AGND
- Q1 pad 1: Earth -> AGND
- Q1 pad 4: Earth -> AGND
- Q2 pad 1: Earth -> AGND
- Q2 pad 4: Earth -> AGND
- Q4 pad 4: Earth -> AGND
- Q5 pad 4: Earth -> AGND
- R1 pad 1: Earth -> AGND
- R10 pad 2: Net-(C88-Pad1) -> /DDR4_x8_32b_1/REFIN
- R11 pad 1: Earth -> /DDR4_x8_32b_1/REFIN
- R11 pad 2: Net-(C88-Pad1) -> AGND
- R116 pad 1: Earth -> AGND
- R117 pad 2: Earth -> AGND
- R156 pad 2: Earth -> AGND
- R2 pad 1: Earth -> AGND
- R23 pad 1: Net-(R23-Pad1) -> +3V3
- R23 pad 2: +3V3 -> Net-(R23-Pad2)
- R27 pad 2: Earth -> AGND
- R28 pad 2: Earth -> AGND
- R29 pad 2: Earth -> AGND
- R3 pad 1: Earth -> AGND
- R30 pad 2: Earth -> AGND
- R33 pad 1: Earth -> AGND
- R39 pad 2: Earth -> AGND
- R4 pad 1: Earth -> AGND
- R41 pad 2: Earth -> AGND
- R5 pad 1: Earth -> AGND
- R53 pad 2: Earth -> AGND
- R54 pad 2: Earth -> AGND
- R55 pad 2: Earth -> AGND
- R56 pad 2: Earth -> AGND
- R57 pad 2: Earth -> AGND
- R58 pad 2: Earth -> AGND
- R59 pad 2: Earth -> AGND
- R6 pad 1: Earth -> AGND
- R61 pad 1: Earth -> AGND
- R7 pad 1: Earth -> AGND
- R70 pad 1: Earth -> AGND
- R71 pad 1: Earth -> AGND
- R8 pad 1: Earth -> AGND
- R88 pad 2: /Ethernet/MX3_N -> Net-(R88-Pad2)
- R9 pad 1: Earth -> AGND
- R92 pad 2: Earth -> AGND
- R93 pad 1: Earth -> AGND
- R94 pad 2: Earth -> AGND
- R95 pad 2: Earth -> AGND
- R96 pad 2: Earth -> AGND
- RS1 pad 1: VMEM -> +1V2
- RS1 pad 2: VDD_DDR_MEM_P -> VDD_DDR_MEM_N
- RS1 pad 3: VDD_DDR_MEM_N -> VDD_DDR_MEM_P
- RS1 pad 4: +1V2 -> VMEM
- RS10 pad 1: VDD_DDRPLL_P -> VDD
- RS10 pad 2: VDD_SOC_CORE_P -> VDD_SOC_CORE_N
- RS10 pad 3: VDD_SOC_CORE_N -> VDD_SOC_CORE_P
- RS10 pad 4: VDD -> VDD_DDRPLL_P
- RS2 pad 1: VCCQ -> VMEM
- RS2 pad 2: VDD_DDR_SOC_N -> VDD_DDR_SOC_P
- RS2 pad 3: VDD_DDR_SOC_P -> VDD_DDR_SOC_N
- RS2 pad 4: VMEM -> VCCQ
- S1 pad 10: Earth -> AGND
- S1 pad 11: Earth -> AGND
- S1 pad 12: Earth -> AGND
- S1 pad 7: Earth -> AGND
- S1 pad 8: Earth -> AGND
- S1 pad 9: Earth -> AGND
- S2 pad 1: Earth -> AGND
- S3 pad 10: Earth -> AGND
- S3 pad 11: Earth -> AGND
- S3 pad 12: Earth -> AGND
- S3 pad 7: Earth -> AGND
- S3 pad 8: Earth -> AGND
- S3 pad 9: Earth -> AGND
- S4 pad 3: Earth -> AGND
- T1 pad 1: /Ethernet/P0_D2_N -> Net-(C199-Pad2)
- T1 pad 11: /Ethernet/P0_D2_N -> /Ethernet/P0_D3_P
- T1 pad 12: /Ethernet/P0_D2_N -> /Ethernet/P0_D3_N
- T1 pad 14: /Ethernet/MX3_N -> /Ethernet/MX4_P
- T1 pad 18: /Ethernet/MX3_N -> Net-(R88-Pad2)
- U1 pad A1: Earth -> AGND
- U1 pad A14: Earth -> AGND
- U1 pad A18: Earth -> AGND
- U1 pad A2: Earth -> AGND
- U1 pad A22: Earth -> AGND
- U1 pad A3: Earth -> AGND
- U1 pad A9: Earth -> AGND
- U1 pad AA2: Earth -> AGND
- U1 pad AB1: Earth -> AGND
- U1 pad AB10: Earth -> AGND
- U1 pad AB13: Earth -> AGND
- U1 pad AB17: Earth -> AGND
- U1 pad AB22: Earth -> AGND
- U1 pad AB4: Earth -> AGND
- U1 pad AB7: Earth -> AGND
- U1 pad D1: Earth -> AGND
- U1 pad D12: Earth -> AGND
- U1 pad E22: Earth -> AGND
- U1 pad E4: Earth -> AGND
- U1 pad F7: Earth -> AGND
- U1 pad G10: Earth -> AGND
- U1 pad G12: Earth -> AGND
- U1 pad G16: Earth -> AGND
- U1 pad G2: Earth -> AGND
- U1 pad G6: Earth -> AGND
- U1 pad G8: Earth -> AGND
- U1 pad H11: Earth -> AGND
- U1 pad H15: Earth -> AGND
- U1 pad H7: Earth -> AGND
- U1 pad H9: Earth -> AGND
- U1 pad J1: Earth -> AGND
- U1 pad J10: Earth -> AGND
- U1 pad J12: Earth -> AGND
- U1 pad J13: Earth -> AGND
- U1 pad J14: Earth -> AGND
- U1 pad J16: Earth -> AGND
- U1 pad J22: Earth -> AGND
- U1 pad J6: Earth -> AGND
- U1 pad J8: Earth -> AGND
- U1 pad K11: Earth -> AGND
- U1 pad K15: Earth -> AGND
- U1 pad K7: Earth -> AGND
- U1 pad K9: Earth -> AGND
- U1 pad L10: Earth -> AGND
- U1 pad L12: Earth -> AGND
- U1 pad L14: Earth -> AGND
- U1 pad L15: Earth -> AGND
- U1 pad L6: Earth -> AGND
- U1 pad L8: Earth -> AGND
- U1 pad M11: Earth -> AGND
- U1 pad M13: Earth -> AGND
- U1 pad M15: Earth -> AGND
- U1 pad M7: Earth -> AGND
- U1 pad N10: Earth -> AGND
- U1 pad N12: Earth -> AGND
- U1 pad N14: Earth -> AGND
- U1 pad N15: Earth -> AGND
- U1 pad N6: Earth -> AGND
- U1 pad N8: Earth -> AGND
- U1 pad P1: Earth -> AGND
- U1 pad P11: Earth -> AGND
- U1 pad P13: Earth -> AGND
- U1 pad P15: Earth -> AGND
- U1 pad P22: Earth -> AGND
- U1 pad P7: Earth -> AGND
- U1 pad P9: Earth -> AGND
- U1 pad R10: Earth -> AGND
- U1 pad R12: Earth -> AGND
- U1 pad R14: Earth -> AGND
- U1 pad R16: Earth -> AGND
- U1 pad R6: Earth -> AGND
- U1 pad R8: Earth -> AGND
- U1 pad T11: Earth -> AGND
- U1 pad T13: Earth -> AGND
- U1 pad T15: Earth -> AGND
- U1 pad T17: Earth -> AGND
- U1 pad T7: Earth -> AGND
- U1 pad T9: Earth -> AGND
- U1 pad U10: Earth -> AGND
- U1 pad U12: Earth -> AGND
- U1 pad U14: Earth -> AGND
- U1 pad U16: Earth -> AGND
- U1 pad U6: Earth -> AGND
- U1 pad U8: Earth -> AGND
- U1 pad V1: Earth -> AGND
- U1 pad V11: Earth -> AGND
- U1 pad V13: Earth -> AGND
- U1 pad V15: Earth -> AGND
- U1 pad V22: Earth -> AGND
- U1 pad V7: Earth -> AGND
- U1 pad V9: Earth -> AGND
- U10 pad A2: Earth -> AGND
- U10 pad A8: Earth -> AGND
- U10 pad A9: Earth -> AGND
- U10 pad C8: Earth -> AGND
- U10 pad D1: Earth -> AGND
- U10 pad D9: Earth -> AGND
- U10 pad E1: Earth -> AGND
- U10 pad E9: Earth -> AGND
- U10 pad G1: Earth -> AGND
- U10 pad G9: Earth -> AGND
- U10 pad H9: Earth -> AGND
- U10 pad K1: Earth -> AGND
- U10 pad K9: Earth -> AGND
- U10 pad N1: Earth -> AGND
- U11 pad 1: Net-(C88-Pad1) -> /DDR4_x8_32b_1/REFIN
- U11 pad 11: Earth -> AGND
- U11 pad 4: Earth -> AGND
- U11 pad 8: Earth -> AGND
- U11 pad 9: +3V3 -> Net-(U11-Pad9)
- U12 pad 10: Earth -> AGND
- U13 pad 1: Earth -> AGND
- U13 pad 10: Earth -> AGND
- U13 pad 11: Earth -> AGND
- U13 pad 13: Earth -> AGND
- U13 pad 14: Net-(R33-Pad2) -> Net-(R23-Pad2)
- U13 pad 15: Earth -> AGND
- U13 pad 25: Earth -> AGND
- U13 pad 35: Earth -> AGND
- U13 pad 47: Earth -> AGND
- U13 pad 5: Earth -> AGND
- U13 pad 51: Earth -> AGND
- U13 pad 6: Net-(R23-Pad1) -> Net-(R33-Pad2)
- U14 pad 2: Earth -> AGND
- U14 pad 3: Earth -> AGND
- U14 pad 9: Earth -> AGND
- U15 pad 2: Earth -> AGND
- U15 pad 3: Earth -> AGND
- U15 pad 9: Earth -> AGND
- U16 pad 14: Earth -> AGND
- U16 pad 15: Earth -> AGND
- U16 pad 17: Earth -> AGND
- U16 pad 6: Earth -> AGND
- U17 pad 2: Earth -> AGND
- U18 pad 10: Earth -> AGND
- U18 pad 11: Earth -> AGND
- U18 pad 12: Earth -> AGND
- U18 pad 13: Earth -> AGND
- U18 pad 14: Earth -> AGND
- U18 pad 19: Earth -> AGND
- U18 pad 23: Earth -> AGND
- U18 pad 29: Earth -> AGND
- U19 pad 2: Earth -> AGND
- U2 pad A2: Earth -> AGND
- U2 pad A8: Earth -> AGND
- U2 pad A9: Earth -> AGND
- U2 pad C8: Earth -> AGND
- U2 pad D1: Earth -> AGND
- U2 pad D9: Earth -> AGND
- U2 pad E1: Earth -> AGND
- U2 pad E9: Earth -> AGND
- U2 pad G1: Earth -> AGND
- U2 pad G9: Earth -> AGND
- U2 pad H9: Earth -> AGND
- U2 pad K1: Earth -> AGND
- U2 pad K9: Earth -> AGND
- U2 pad N1: Earth -> AGND
- U20 pad 3: Earth -> AGND
- U21 pad 3: Earth -> AGND
- U22 pad 3: Earth -> AGND
- U23 pad 3: Earth -> AGND
- U24 pad 3: Earth -> AGND
- U25 pad 3: Earth -> AGND
- U26 pad 13: Earth -> AGND
- U27 pad 15: Earth -> AGND
- U27 pad 16: Earth -> AGND
- U27 pad 17: Earth -> AGND
- U27 pad 5: Earth -> AGND
- U27 pad 6: Earth -> AGND
- U27 pad 7: Earth -> AGND
- U27 pad 8: Earth -> AGND
- U28 pad 3: Earth -> AGND
- U29 pad 3: Earth -> AGND
- U3 pad A2: Earth -> AGND
- U3 pad A8: Earth -> AGND
- U3 pad A9: Earth -> AGND
- U3 pad C8: Earth -> AGND
- U3 pad D1: Earth -> AGND
- U3 pad D9: Earth -> AGND
- U3 pad E1: Earth -> AGND
- U3 pad E9: Earth -> AGND
- U3 pad G1: Earth -> AGND
- U3 pad G9: Earth -> AGND
- U3 pad H9: Earth -> AGND
- U3 pad K1: Earth -> AGND
- U3 pad K9: Earth -> AGND
- U3 pad N1: Earth -> AGND
- U30 pad 3: Earth -> AGND
- U31 pad 3: Earth -> AGND
- U32 pad 3: Earth -> AGND
- U33 pad 3: Earth -> AGND
- U35 pad 2: Earth -> AGND
- U35 pad 7: Earth -> AGND
- U36 pad 5: Earth -> AGND
- U36 pad 7: Earth -> AGND
- U37 pad 3: Earth -> AGND
- U38 pad 3: Earth -> AGND
- U4 pad A2: Earth -> AGND
- U4 pad A8: Earth -> AGND
- U4 pad A9: Earth -> AGND
- U4 pad C8: Earth -> AGND
- U4 pad D1: Earth -> AGND
- U4 pad D9: Earth -> AGND
- U4 pad E1: Earth -> AGND
- U4 pad E9: Earth -> AGND
- U4 pad G1: Earth -> AGND
- U4 pad G9: Earth -> AGND
- U4 pad H9: Earth -> AGND
- U4 pad K1: Earth -> AGND
- U4 pad K9: Earth -> AGND
- U4 pad N1: Earth -> AGND
- U49 pad 3: Earth -> AGND
- U49 pad 4: Earth -> AGND
- U5 pad A2: Earth -> AGND
- U5 pad A8: Earth -> AGND
- U5 pad A9: Earth -> AGND
- U5 pad C8: Earth -> AGND
- U5 pad D1: Earth -> AGND
- U5 pad D9: Earth -> AGND
- U5 pad E1: Earth -> AGND
- U5 pad E9: Earth -> AGND
- U5 pad G1: Earth -> AGND
- U5 pad G9: Earth -> AGND
- U5 pad H9: Earth -> AGND
- U5 pad K1: Earth -> AGND
- U5 pad K9: Earth -> AGND
- U5 pad N1: Earth -> AGND
- U50 pad 2: Earth -> AGND
- U50 pad 3: Earth -> AGND
- U50 pad 9: Earth -> AGND
- U6 pad A2: Earth -> AGND
- U6 pad A8: Earth -> AGND
- U6 pad A9: Earth -> AGND
- U6 pad C8: Earth -> AGND
- U6 pad D1: Earth -> AGND
- U6 pad D9: Earth -> AGND
- U6 pad E1: Earth -> AGND
- U6 pad E9: Earth -> AGND
- U6 pad G1: Earth -> AGND
- U6 pad G9: Earth -> AGND
- U6 pad H9: Earth -> AGND
- U6 pad K1: Earth -> AGND
- U6 pad K9: Earth -> AGND
- U6 pad N1: Earth -> AGND
- U7 pad A2: Earth -> AGND
- U7 pad A8: Earth -> AGND
- U7 pad A9: Earth -> AGND
- U7 pad C8: Earth -> AGND
- U7 pad D1: Earth -> AGND
- U7 pad D9: Earth -> AGND
- U7 pad E1: Earth -> AGND
- U7 pad E9: Earth -> AGND
- U7 pad G1: Earth -> AGND
- U7 pad G9: Earth -> AGND
- U7 pad H9: Earth -> AGND
- U7 pad K1: Earth -> AGND
- U7 pad K9: Earth -> AGND
- U7 pad N1: Earth -> AGND
- U8 pad A2: Earth -> AGND
- U8 pad A8: Earth -> AGND
- U8 pad A9: Earth -> AGND
- U8 pad C8: Earth -> AGND
- U8 pad D1: Earth -> AGND
- U8 pad D9: Earth -> AGND
- U8 pad E1: Earth -> AGND
- U8 pad E9: Earth -> AGND
- U8 pad G1: Earth -> AGND
- U8 pad G9: Earth -> AGND
- U8 pad H9: Earth -> AGND
- U8 pad K1: Earth -> AGND
- U8 pad K9: Earth -> AGND
- U8 pad N1: Earth -> AGND
- U9 pad A2: Earth -> AGND
- U9 pad A8: Earth -> AGND
- U9 pad A9: Earth -> AGND
- U9 pad C8: Earth -> AGND
- U9 pad D1: Earth -> AGND
- U9 pad D9: Earth -> AGND
- U9 pad E1: Earth -> AGND
- U9 pad E9: Earth -> AGND
- U9 pad G1: Earth -> AGND
- U9 pad G9: Earth -> AGND
- U9 pad H9: Earth -> AGND
- U9 pad K1: Earth -> AGND
- U9 pad K9: Earth -> AGND
- U9 pad N1: Earth -> AGND
- X1 pad 2: Earth -> AGND
- X2 pad 2: Earth -> AGND
- Y1 pad 2: Earth -> AGND
- Y2 pad 2: Earth -> AGND
- Y3 pad 2: Earth -> AGND
Routing:
- net AGND: track 0.00 -> 760.2 mm, vias 0 -> 494
- net +1V2: track 0.00 -> 228.2 mm, vias 0 -> 102
- net VD: track 0.00 -> 200.9 mm, vias 0 -> 11
- net VDD_DDR_VPP_N: track 0.00 -> 85.3 mm, vias 0 -> 17
- net /Power.sch/PWR_ON: track 0.00 -> 69.1 mm, vias 0 -> 1
- net DDR_DM2: track 0.00 -> 62.0 mm, vias 0 -> 2
- net DDR_DQ16: track 0.00 -> 61.9 mm, vias 0 -> 2
- net DDR_DQ19: track 0.00 -> 61.9 mm, vias 0 -> 2
- net DDR_DQ22: track 0.00 -> 60.1 mm, vias 0 -> 2
- net DDR_DQ20: track 0.00 -> 60.0 mm, vias 0 -> 2
- net VDD_GIVDD_P: track 0.00 -> 58.8 mm, vias 0 -> 34
- net DDR_DQ18: track 0.00 -> 58.8 mm, vias 0 -> 2
- net DDR_DQS2_N: track 0.00 -> 58.4 mm, vias 0 -> 2
- net DDR_DQS2_P: track 0.00 -> 57.9 mm, vias 0 -> 2
- net DDR_DQ17: track 0.00 -> 57.2 mm, vias 0 -> 2
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- added copper zone on F.Cu, net +12V
- added copper zone on In3.Cu, net +12V
- added copper zone on In1.Cu, net +1V0
- added copper zone on F.Cu, net +1V2
- added copper zone on In8.Cu, net +1V2
- added copper zone on In1.Cu, net +2V5
- added copper zone on F.Cu, net +5V
- added copper zone on F.Cu, net AGND
- added copper zone on In1.Cu, net AGND
- added copper zone on F.Cu, net AVDD_DDRPLL_P
- added copper zone on F.Cu, net Net-(C146-Pad1)
- added copper zone on In2.Cu, net Net-(C181-Pad1)
- added copper zone on F.Cu, net Net-(D7-Pad2)
- added copper zone on F.Cu, net Net-(J9-PadC35)
- added copper zone on F.Cu, net Net-(L1-Pad1)
- added copper zone on F.Cu, net Net-(L3-Pad1)
- added copper zone on F.Cu, net Net-(L4-Pad1)
- added copper zone on F.Cu, net Net-(L6-Pad1)
- added copper zone on F.Cu, net VAA
- added copper zone on F.Cu, net VDD_DDRPLL_P
- added copper zone on F.Cu, net VDD_DDR_VPP_P
- added copper zone on F.Cu, net VDD_GIVDD_P
- added copper zone on In1.Cu, net VDD_GIVDD_P
- added copper zone on In2.Cu, net VDD_GIVDD_P
- added copper zone on F.Cu, net VMEM
Other:
- outline, holes or cut-outs redrawn
- copper layers 2 -> 10
- net class 0,0762 added: clearance 0.0762, trace_width 0.0762, via_dia 0.3556, via_drill 0.2032
- net class 0,12192 added: clearance 0.0762, trace_width 0.12192, via_dia 0.3556, via_drill 0.2032
- net class 0,1524 added: clearance 0.0762, trace_width 0.1524, via_dia 0.3556, via_drill 0.2032
- net class 0,2032 added: clearance 0.0762, trace_width 0.2032, via_dia 0.3556, via_drill 0.2032
- net class 0,254 added: clearance 0.0762, trace_width 0.254, via_dia 0.3556, via_drill 0.2032
- net class Default: clearance 0.2 -> 0.0762; trace_width 0.25 -> 0.0762; via_dia 0.8 -> 0.3556; via_drill 0.4 -> 0.2032
- net class temp added: clearance 0.2, trace_width 0.25, via_dia 0.881, via_drill 0.635
- rule trace_clearance: 0.2 -> 0.0762
- rule trace_min: 0.2 -> 0.0762
- rule via_min_drill: 0.3 -> 0.2032
- rule via_min_size: 0.4 -> 0.3556

Commit message: Update kicad electric lines
Parts:
- moved J19 5.56 mm to (68.1, 46.0), turned to 270 degrees
Routing:
- net DDR_ACT_N: track 17.7 -> 172.0 mm
- net DDR_CKE: track 21.4 -> 166.8 mm
- net DDR_A1: track 20.3 -> 156.2 mm
- net DDR_BG0: track 28.0 -> 163.1 mm
- net DDR_ODT: track 18.1 -> 148.9 mm
- net DDR_CKE1: track 30.7 -> 147.9 mm
- net DDR_BG1: track 22.2 -> 123.2 mm
- net DDR_CS0_N: track 19.9 -> 112.9 mm
- net DDR_ODT1: track 26.8 -> 102.7 mm
- net CHIPLINK_RX_DAT7: track 0.58 -> 74.0 mm, vias 1 -> 2
- net CHIPLINK_RX_DAT12: track 1.55 -> 74.0 mm
- net CHIPLINK_RX_DAT3: track 1.48 -> 73.4 mm
- net CHIPLINK_RX_DAT6: track 1.46 -> 70.0 mm
- net DDR_A3: track 18.5 -> 86.5 mm
- net CHIPLINK_RX_DAT1: track 4.36 -> 70.0 mm
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